Commit message: Refactor for noetic

File: urdf/braccio_arm.urdf (robot description, URDF)
Before this commit: robot visual, 8 links, 7 joints
Links:
- link braccio_base_link: geometry visual mesh filename=package://braccio_manipulator/stl/braccio_base.stl scale=0.001 0.001 0.001
- link elbow_link: geometry visual mesh filename=package://braccio_manipulator/stl/braccio_elbow.stl scale=0.001 0.001 0.001
- link left_gripper_link: geometry visual mesh filename=package://braccio_manipulator/stl/braccio_left_gripper.stl scale=0.001 0.001 0.001
- link right_gripper_link: geometry visual mesh filename=package://braccio_manipulator/stl/braccio_right_gripper.stl scale=0.001 0.001 0.001
- link shoulder_link: geometry visual mesh filename=package://braccio_manipulator/stl/braccio_shoulder.stl scale=0.001 0.001 0.001
- link wrist_pitch_link: geometry visual mesh filename=package://braccio_manipulator/stl/braccio_wrist_pitch.stl scale=0.001 0.001 0.001
- link wrist_roll_link: geometry visual mesh filename=package://braccio_manipulator/stl/braccio_wrist_roll.stl scale=0.001 0.001 0.001

Commit message: Added hardware interface, has error with soft limits

File: urdf/braccio_arm.urdf (robot description, URDF)
Before this commit: robot visual, 8 links, 7 joints
Joints:
- joint base_joint: limit lower=0.0 upper=3.1416 effort=1000.0 velocity=1.0 -> lower=$(eval -pi/2) upper=$(eval pi/2) effort=1000.0 velocity=10.0
- joint elbow_joint: limit lower=0 upper=3.1416 effort=1000.0 velocity=1.0 -> lower=$(eval -pi/2) upper=$(eval pi/2) effort=1000.0 velocity=10.0; origin xyz=0 0 0.125 rpy=${-pi/2} 0 0 -> xyz=0 0 0.125 rpy=0 0 0
- joint shoulder_joint: limit lower=0.2618 upper=2.8798 effort=1000.0 velocity=1.0 -> lower=$(eval -5*pi/12) upper=$(eval 5*pi/12) effort=1000.0 velocity=10.0; origin xyz=0 -0.002 0.072 rpy=${-pi/2} 0 0 -> xyz=0 -0.002 0.072 rpy=0 0 0
- joint wrist_pitch_joint: limit lower=0 upper=3.1416 effort=1000.0 velocity=1.0 -> lower=$(eval -pi/2) upper=$(eval pi/2) effort=1000.0 velocity=10.0; origin xyz=0 0 0.125 rpy=${-pi/2} 0 0 -> xyz=0 0 0.125 rpy=0 0 0
- joint wrist_roll_joint: limit lower=0.0 upper=3.1416 effort=1000.0 velocity=1.0 -> lower=$(eval -pi/2) upper=$(eval 35*pi/180) effort=1000.0 velocity=10.0; origin xyz=0 0.0 0.06 rpy=0 0 0 -> xyz=0 0.0 0.06 rpy=0 0 $(eval -pi/2)
